File: Rev_1/ECAD/Display/display.kicad_sch (KiCad schematic)
At the start: 2 parts, among them J1 Conn_01x16_Socket, J2 Conn_01x16_Socket

Commit message: Mostly finished
Parts:
- J1: Part-DB ID (none) -> 65
Changed lines of the file:
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@@
+			)
+		)
+		(property "Part-DB ID" ""
+			(at 142.24 109.22 0)
+			(hide yes)
+			(show_name no)
+			(do_not_autoplace no)
+			(effects
+				(font
+					(size 1.27 1.27)
+				)
 			)
 		)
@@
 			(at 93.98 109.22 0)
 			(hide yes)
+			(show_name no)
+			(do_not_autoplace no)
+			(effects
+				(font
+					(size 1.27 1.27)
+				)
+			)
+		)
+		(property "Part-DB ID" "65"
+			(at 93.98 109.22 0)
+			(hide yes)
