File: Rev_1/ECAD/Driver/_autosave-driver.kicad_pcb (KiCad board)
At the start: 4 copper layers, 40.6 x 46 mm, 62 parts, among them J1 USB_C_Receptacle_USB2.0_16P, J2 Conn_ARM_JTAG_SWD_10, J4 Conn_01x16_Pin, J5 Conn_01x16_Pin, Q1 NPN, Q10 PMOS, Q11 PMOS, Q12 PMOS, Q13 PMOS, Q14 PMOS, Q15 PMOS, Q16 PMOS, Q17 PMOS, Q2 PMOS, Q3 PMOS, Q4 PMOS, Q5 PMOS, Q6 PMOS, Q7 PMOS, Q8 PMOS, Q9 PMOS, U1 STM32C551KET6, U2 USBLC6-2SC6, U3 25CSM04xxSN, U4 TPS62A01ADRL, U5 74HC595, U6 74HC595, U7 TLC59283DBQR, Y1 8MHz

Commit message: Mostly finished
Changed lines of the file:
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@@
 		(tags "resistor")
 		(property "Reference" "R5"
-			(at -0.952 1.191501 0)
+			(at 1.1552 -1.267701 0)
 			(layer "F.SilkS")
 			(effects
@@
 		(tags "resistor handsolder")
 		(property "Reference" "R7"
-			(at 2.159001 -0.000001 0)
+			(at 2.133601 0.380999 0)
 			(layer "F.SilkS")
 			(effects
