File: Rev_1/ECAD/Driver/driver.kicad_sch (KiCad schematic)
At the start: 34 parts, among them J3 USB_C_Receptacle_USB2.0_16P, J5 Conn_ARM_JTAG_SWD_10, Q17 NPN, U1 25CSM04xxSN, U2 STM32C551KET6, U22 USBLC6-2SC6, U3 TPS62A01ADRL, Y1 8MHz

Commit message: Mostly finished
Parts:
- removed Q17: NPN, Package_TO_SOT_SMD:SOT-23, symbol Simulation_SPICE:NPN
- added Q1: NPN, symbol filip:NPN_Alternative_1
- BZ1: Part-DB ID (none) -> 71
- C1: renamed from C10; Part-DB ID (none) -> 88
- C10: renamed from C9; Part-DB ID (none) -> 9
- C11: renamed from C13; Part-DB ID (none) -> 26
- C12: renamed from C2; Part-DB ID (none) -> 86
- C13: renamed from C3; Part-DB ID (none) -> 5
- C2: renamed from C11; Part-DB ID (none) -> 88
- C3: renamed from C16; Part-DB ID (none) -> 76
- C4: renamed from C14; Part-DB ID (none) -> 9
- C5: Part-DB ID (none) -> 87
- C6: renamed from C15; Part-DB ID (none) -> 9
- C7: renamed from C8; Part-DB ID (none) -> 9
- C8: renamed from C12; Part-DB ID (none) -> 9
- C9: renamed from C1; Part-DB ID (none) -> 26
- D1: Part-DB ID (none) -> 49
- FB1: Part-DB ID (none) -> 51
- J1: renamed from J3; Part-DB ID (none) -> 82
- J2: renamed from J5; Part-DB ID (none) -> 85
- L1: Part-DB ID (none) -> 83
- R1: renamed from R7; Part-DB ID (none) -> 17
- R2: renamed from R8; Part-DB ID (none) -> 17
- R3: renamed from R13; Part-DB ID (none) -> 67
- R4: renamed from R5; Part-DB ID (none) -> 67
- R5: renamed from R9; Part-DB ID (none) -> 72
- R6: renamed from R4; Part-DB ID (none) -> 67
- R7: renamed from R2; Part-DB ID (none) -> 73
- R8: renamed from R3; Part-DB ID (none) -> 14
- TH1: Part-DB ID (none) -> 74
- U1: renamed from U2; Part-DB ID (none) -> 77
- U3: renamed from U1; Part-DB ID (none) -> 79
- U4: renamed from U3; Part-DB ID (none) -> 78
- Y1: Part-DB ID (none) -> 89
- renumbered U22 to U2
Connections:
- net GND: now also Q1.2 (E)
- net at R5.2: now also Q1.1 (B)
- net at BZ1.2 (-): now also Q1.3 (C)
