File: Rev_1/ECAD/Driver/row_col_driver.kicad_sch (KiCad schematic)
At the start: 27 parts, among them J1 Conn_01x16_Pin, J2 Conn_01x16_Pin, J4 Conn_02x05_Counter_Clockwise, Q1 PMOS, Q10 PMOS, Q11 PMOS, Q12 PMOS, Q13 PMOS, Q14 PMOS, Q15 PMOS, Q16 PMOS, Q2 PMOS, Q3 PMOS, Q4 PMOS, Q5 PMOS, Q6 PMOS, Q7 PMOS, Q8 PMOS, Q9 PMOS, U4 TLC59283DBQR, U5 74HC595, U6 74HC595

Commit message: Mostly finished
Parts:
- removed J4: Conn_02x05_Counter_Clockwise, symbol Connector_Generic:Conn_02x05_Counter_Clockwise
- removed Q1, Q10, Q11, Q12, Q13, Q14, Q15, Q16, Q2, Q3, Q4, Q5, Q6, Q7, Q8, Q9: PMOS, Package_TO_SOT_SMD:SOT-23, symbol Simulation_SPICE:PMOS
- added Q10, Q11, Q12, Q13, Q14, Q15, Q16, Q17, Q2, Q3, Q4, Q5, Q6, Q7, Q8, Q9: PMOS, Package_TO_SOT_SMD:SOT-23, symbol filip:PMOS_Alternative_1
- C14: renamed from C6; Part-DB ID (none) -> 9
- C15: renamed from C7; Part-DB ID (none) -> 9
- C16: renamed from C4; Part-DB ID (none) -> 9
- J4: renamed from J2; Part-DB ID (none) -> 84
- J5: renamed from J1; Part-DB ID (none) -> 84
- R10: renamed from R1; Part-DB ID (none) -> 72
- R9: renamed from R6; Part-DB ID (none) -> 70
- U5, U6: Part-DB ID (none) -> 81
- U7: renamed from U4; Part-DB ID (none) -> 80
Connections:
- net +3V3: now also Q10.2 (S), Q11.2 (S), Q12.2 (S), Q13.2 (S), Q14.2 (S), Q15.2 (S), Q16.2 (S), Q17.2 (S), Q2.2 (S), Q3.2 (S), Q4.2 (S), Q5.2 (S), Q6.2 (S), Q7.2 (S), Q8.2 (S), Q9.2 (S)
- net ROW0: now also Q2.3 (D)
- net ROW0_G: now also Q2.1 (G)
- net ROW1: now also Q3.3 (D)
- net ROW10: now also Q12.3 (D)
- net ROW10_G: now also Q12.1 (G)
- net ROW11: now also Q13.3 (D)
- net ROW11_G: now also Q13.1 (G)
- net ROW12: now also Q14.3 (D)
- net ROW12_G: now also Q14.1 (G)
- net ROW13: now also Q15.3 (D)
- net ROW13_G: now also Q15.1 (G)
- net ROW14: now also Q16.3 (D)
- net ROW14_G: now also Q16.1 (G)
- net ROW15: now also Q17.3 (D)
- net ROW15_G: now also Q17.1 (G)
- net ROW1_G: now also Q3.1 (G)
- net ROW2: now also Q4.3 (D)
- net ROW2_G: now also Q4.1 (G)
- net ROW3: now also Q5.3 (D)
- net ROW3_G: now also Q5.1 (G)
- net ROW4: now also Q6.3 (D)
- net ROW4_G: now also Q6.1 (G)
- net ROW5: now also Q7.3 (D)
- net ROW5_G: now also Q7.1 (G)
- net ROW6: now also Q8.3 (D)
- net ROW6_G: now also Q8.1 (G)
- net ROW7: now also Q9.3 (D)
- net ROW7_G: now also Q9.1 (G)
- net ROW8: now also Q10.3 (D)
- net ROW8_G: now also Q10.1 (G)
- net ROW9: now also Q11.3 (D)
- net ROW9_G: now also Q11.1 (G)
